File: pd-buddy-sink/voltage_regulator.sch (KiCad schematic (older format))
At the start: 5 parts, among them U1 AP2204R-3.3TRG1

Commit message: Update footprints
The SOT-89 footprint changed its name slightly in the KiCad library,
so the voltage regulator has been updated accordingly.  It has a nice
new 3D model too.  It's not weird and blue anymore.  I like it.

The SOD-123 was also updated to have a 3D model.  The board now only
lacks models for the footprints I made myself.  Heh.
Parts:
- U1: footprint TO_SOT_Packages_SMD:SOT89-3_Housing -> TO_SOT_Packages_SMD:SOT-89-3
Changed lines of the file:
@@
-$EndComp
-$Comp
-L AP2204R-3.3TRG1 U1
-U 1 1 588FA408
-P 6050 3500
-F 0 "U1" H 6250 3200 60  0000 C CNN
-F 1 "AP2204R-3.3TRG1" H 6050 3700 60  0000 C CNN
-F 2 "TO_SOT_Packages_SMD:SOT89-3_Housing" H 6150 3100 60  0001 C CNN
-F 3 "http://www.diodes.com/_files/datasheets/AP2204.pdf" H 6250 3200 60  0001 C CNN
-	1    6050 3500
-	1    0    0    -1
 $EndComp
 $Comp
@@
 Wire Wire Line
 	4500 3800 4500 3900
+$Comp
+L AP2204R-3.3TRG1 U1
+U 1 1 592B31D5
+P 6050 3500
+F 0 "U1" H 6250 3200 60  0000 C CNN
+F 1 "AP2204R-3.3TRG1" H 6050 3700 60  0000 C CNN
+F 2 "TO_SOT_Packages_SMD:SOT-89-3" H 6150 3100 60  0001 C CNN
+F 3 "http://www.diodes.com/_files/datasheets/AP2204.pdf" H 6250 3200 60  0001 C CNN
+	1    6050 3500
+	1    0    0    -1
+$EndComp
 $EndSCHEMATC
