File: pd-buddy-sink/microcontroller.sch (KiCad schematic (older format))
At the start: 20 parts, among them P1 SWD, SW1 Boot, SW2 Setup, U2 STM32F072C8Ux

Commit message: Use PTS810 pushbutton switch for SW2
Assuming I'm going to keep ordering boards from MacroFab, it makes sense
to use their house parts as much as possible.  Therefore, the next
boards will use a C&K PTS810 as the Setup switch instead of an Alps
SKQG.  In addition to saving money, this change allows room for larger
"Setup" and "GND" labels.
Parts:
- SW2: footprint Buttons_Switches_SMD:SW_SPST_SKQG -> Buttons_Switches_SMD:SW_SPST_PTS810
Changed lines of the file:
@@
 Title "PD Buddy Sink"
 Date ""
-Rev "0.3"
+Rev "1.0"
 Comp ""
 Comment1 ""
@@
 F 0 "SW2" H 6850 5950 50  0000 L CNN
 F 1 "Setup" H 6800 5790 50  0000 C CNN
-F 2 "Buttons_Switches_SMD:SW_SPST_SKQG" H 6800 6050 50  0001 C CNN
+F 2 "Buttons_Switches_SMD:SW_SPST_PTS810" H 6800 6050 50  0001 C CNN
 F 3 "" H 6800 6050 50  0000 C CNN
 	1    6800 5850
