File: pd-buddy-sink/microcontroller.sch (KiCad schematic (older format))
At the start: 20 parts, among them P1 SWD, SW1 Boot, SW2 Setup, U2 STM32F072C8Ux

Commit message: Changed SW1 and P1 footprints
The components on the bottom, SW1 and P1, were using slightly modified
footprints from the KiCad library (default, but with no paste on any
pads) in v0.3.  Now they're back to the default footprints, but with
local paste clearance set to -100% to make sure there's no paste on any
of their pads.
Parts:
- P1: footprint pd-buddy:Pin_Header_Straight_2x05_Pitch1.27mm_SMD_NOPASTE -> Pin_Headers:Pin_Header_Straight_2x05_Pitch1.27mm_SMD
- SW1: footprint pd-buddy:SW_SPDT_PCM12_NOPASTE -> Buttons_Switches_SMD:SW_SPDT_PCM12
Changed lines of the file:
@@
 F 0 "SW1" H 1100 1520 50  0000 C CNN
 F 1 "Boot" H 1100 1150 50  0000 C CNN
-F 2 "pd-buddy:SW_SPDT_PCM12_NOPASTE" H 1100 1350 50  0001 C CNN
+F 2 "Buttons_Switches_SMD:SW_SPDT_PCM12" H 1100 1350 50  0001 C CNN
 F 3 "" H 1100 1350 50  0000 C CNN
 	1    1100 1350
@@
 F 0 "P1" H 4850 6500 50  0000 C CNN
 F 1 "SWD" H 4850 5900 50  0000 C CNN
-F 2 "pd-buddy:Pin_Header_Straight_2x05_Pitch1.27mm_SMD_NOPASTE" H 4850 5000 50  0001 C CNN
+F 2 "Pin_Headers:Pin_Header_Straight_2x05_Pitch1.27mm_SMD" H 4850 5000 50  0001 C CNN
 F 3 "" H 4850 5000 50  0000 C CNN
 	1    4850 6200

Commit message: Added test points, replaced SW1 with R11
More test points will be needed for automated testing, so I've added the
first two I know of.

With firmware version 1.2.0+, there's not much reason to install SW1
anymore.  This commit replaces it with R11, an unpopulated resistor
footprint that does the same thing as bridging the two pins of SW1 used
to do, just in case an upgrade make the `boot` command stop working.
Parts:
- removed P1: SWD, Pin_Headers:Pin_Header_Straight_2x05_Pitch1.27mm_SMD, symbol CONN_02X05
- removed SW1: Boot, Buttons_Switches_SMD:SW_SPDT_PCM12, symbol SW_SPDT
- added P1: SWD, Pin_Headers:Pin_Header_Straight_2x05_Pitch1.27mm_SMD, symbol Conn_02x05_Odd_Even
- added R11: 0Ω, Resistors_SMD:R_0402, symbol R
- added TP3: Setup, Measurement_Points:Measurement_Point_Round-SMD-Pad_Small, symbol Test_Point
Connections:
- net +3V3: now also P1.1 (Pin_1), R11.1
- net BOOT: now also R11.2
- net GND: now also P1.3 (Pin_3), P1.5 (Pin_5), P1.9 (Pin_9)
- net SWCLK: now also P1.4 (Pin_4)
- net SWDIO: now also P1.2 (Pin_2)
- net nRST: now also P1.10 (Pin_10)
- net at R5.1, R6.1, SW2.2: now also TP3.1
Changed lines of the file:
@@
 D-
-$Comp
-L SW_SPDT SW1
-U 1 1 589013E6
-P 1100 1350
-F 0 "SW1" H 1100 1520 50  0000 C CNN
-F 1 "Boot" H 1100 1150 50  0000 C CNN
-F 2 "Buttons_Switches_SMD:SW_SPDT_PCM12" H 1100 1350 50  0001 C CNN
-F 3 "" H 1100 1350 50  0000 C CNN
-	1    1100 1350
-	0    -1   -1   0
-$EndComp
 $Comp
 L R R2
@@
 L +3.3V #PWR08
 U 1 1 5890170D
-P 1200 1150
-F 0 "#PWR08" H 1200 1000 50  0001 C CNN
-F 1 "+3.3V" H 1200 1290 50  0000 C CNN
-F 2 "" H 1200 1150 50  0000 C CNN
-F 3 "" H 1200 1150 50  0000 C CNN
-	1    1200 1150
+P 1100 1300
+F 0 "#PWR08" H 1100 1150 50  0001 C CNN
+F 1 "+3.3V" H 1100 1440 50  0000 C CNN
+F 2 "" H 1100 1300 50  0000 C CNN
+F 3 "" H 1100 1300 50  0000 C CNN
+	1    1100 1300
 	1    0    0    -1
 $EndComp
 $Comp
 L GND #PWR09
-U 1 1 58901727
-P 700 1150
-F 0 "#PWR09" H 700 900 50  0001 C CNN
-F 1 "GND" H 700 1000 50  0000 C CNN
-F 2 "" H 700 1150 50  0000 C CNN
-F 3 "" H 700 1150 50  0000 C CNN
-	1    700  1150
-	1    0    0    -1
-$EndComp
-$Comp
-L GND #PWR010
 U 1 1 58901B1C
 P 5700 5000
-F 0 "#PWR010" H 5700 4750 50  0001 C CNN
+F 0 "#PWR09" H 5700 4750 50  0001 C CNN
 F 1 "GND" H 5700 4850 50  0000 C CNN
 F 2 "" H 5700 5000 50  0000 C CNN
@@
 $EndComp
 $Comp
-L +3.3V #PWR011
+L +3.3V #PWR010
 U 1 1 5891514A
 P 2000 2000
-F 0 "#PWR011" H 2000 1850 50  0001 C CNN
+F 0 "#PWR010" H 2000 1850 50  0001 C CNN
 F 1 "+3.3V" H 2000 2140 50  0000 C CNN
 F 2 "" H 2000 2000 50  0000 C CNN
@@
 $EndComp
 $Comp
-L +3.3V #PWR012
+L +3.3V #PWR011
 U 1 1 58915182
 P 5700 900
-F 0 "#PWR012" H 5700 750 50  0001 C CNN
+F 0 "#PWR011" H 5700 750 50  0001 C CNN
 F 1 "+3.3V" H 5700 1040 50  0000 C CNN
 F 2 "" H 5700 900 50  0000 C CNN
@@
 $EndComp
 $Comp
-L GND #PWR013
+L GND #PWR012
 U 1 1 58915422
 P 1300 1600
-F 0 "#PWR013" H 1300 1350 50  0001 C CNN
+F 0 "#PWR012" H 1300 1350 50  0001 C CNN
 F 1 "GND" H 1300 1450 50  0000 C CNN
 F 2 "" H 1300 1600 50  0000 C CNN
@@
 $EndComp
 $Comp
-L +3.3V #PWR014
+L +3.3V #PWR013
 U 1 1 58916B17
 P 1600 6000
-F 0 "#PWR014" H 1600 5850 50  0001 C CNN
+F 0 "#PWR013" H 1600 5850 50  0001 C CNN
 F 1 "+3.3V" H 1600 6140 50  0000 C CNN
 F 2 "" H 1600 6000 50  0000 C CNN
@@
 $EndComp
 $Comp
-L GND #PWR015
+L GND #PWR014
 U 1 1 58916B2E
 P 1600 6700
-F 0 "#PWR015" H 1600 6450 50  0001 C CNN
+F 0 "#PWR014" H 1600 6450 50  0001 C CNN
 F 1 "GND" H 1600 6550 50  0000 C CNN
 F 2 "" H 1600 6700 50  0000 C CNN
@@
 $EndComp
 $Comp
-L +3.3V #PWR016
+L +3.3V #PWR015
 U 1 1 58924A22
 P 1100 3300
-F 0 "#PWR016" H 1100 3150 50  0001 C CNN
+F 0 "#PWR015" H 1100 3150 50  0001 C CNN
 F 1 "+3.3V" H 1100 3440 50  0000 C CNN
 F 2 "" H 1100 3300 50  0000 C CNN
@@
 $EndComp
 $Comp
-L +3.3V #PWR017
+L +3.3V #PWR016
 U 1 1 58928192
 P 6800 5300
-F 0 "#PWR017" H 6800 5150 50  0001 C CNN
+F 0 "#PWR016" H 6800 5150 50  0001 C CNN
 F 1 "+3.3V" H 6800 5440 50  0000 C CNN
 F 2 "" H 6800 5300 50  0000 C CNN
@@
 $EndComp
 $Comp
-L GND #PWR018
+L GND #PWR017
 U 1 1 5892882F
 P 6800 6500
-F 0 "#PWR018" H 6800 6250 50  0001 C CNN
+F 0 "#PWR017" H 6800 6250 50  0001 C CNN
 F 1 "GND" H 6800 6350 50  0000 C CNN
 F 2 "" H 6800 6500 50  0000 C CNN
@@
 NoConn ~ 9700 3800
 $Comp
-L CONN_02X05 P1
-U 1 1 5892D0FE
-P 4850 6200
-F 0 "P1" H 4850 6500 50  0000 C CNN
-F 1 "SWD" H 4850 5900 50  0000 C CNN
-F 2 "Pin_Headers:Pin_Header_Straight_2x05_Pitch1.27mm_SMD" H 4850 5000 50  0001 C CNN
-F 3 "" H 4850 5000 50  0000 C CNN
-	1    4850 6200
-	1    0    0    -1
-$EndComp
-$Comp
-L GND #PWR019
+L GND #PWR018
 U 1 1 5892D636
 P 4500 6500
-F 0 "#PWR019" H 4500 6250 50  0001 C CNN
+F 0 "#PWR018" H 4500 6250 50  0001 C CNN
 F 1 "GND" H 4500 6350 50  0000 C CNN
 F 2 "" H 4500 6500 50  0000 C CNN
@@
 $EndComp
 $Comp
-L +3.3V #PWR020
+L +3.3V #PWR019
 U 1 1 5892D6D6
 P 4500 5900
-F 0 "#PWR020" H 4500 5750 50  0001 C CNN
+F 0 "#PWR019" H 4500 5750 50  0001 C CNN
 F 1 "+3.3V" H 4500 6040 50  0000 C CNN
 F 2 "" H 4500 5900 50  0000 C CNN
@@
 	9700 4100 10000 4100
 Wire Wire Line
-	1100 1550 1100 1900
+	1100 1700 1100 1900
 Wire Wire Line
 	1100 1800 2100 1800
-Wire Wire Line
-	700  1150 700  1050
-Wire Wire Line
-	700  1050 1000 1050
-Wire Wire Line
-	1000 1050 1000 1150
 Wire Wire Line
 	6000 4900 6000 4800
@@
 	6800 5800 6800 6000
 Wire Wire Line
-	6700 5900 6800 5900
+	6700 5900 6900 5900
 Connection ~ 6800 5900
 Wire Wire Line
@@
 	10000 4400 10000 4500
 $Comp
-L GND #PWR021
+L GND #PWR020
 U 1 1 589313D4
 P 10000 5300
-F 0 "#PWR021" H 10000 5050 50  0001 C CNN
+F 0 "#PWR020" H 10000 5050 50  0001 C CNN
 F 1 "GND" H 10000 5150 50  0000 C CNN
 F 2 "" H 10000 5300 50  0000 C CNN
@@
 Connection ~ 1100 1800
 $Comp
-L GND #PWR022
+L GND #PWR021
 U 1 1 58B996F4
 P 1100 2300
-F 0 "#PWR022" H 1100 2050 50  0001 C CNN
+F 0 "#PWR021" H 1100 2050 50  0001 C CNN
 F 1 "GND" H 1100 2150 50  0000 C CNN
 F 2 "" H 1100 2300 50  0000 C CNN
@@
 	6100 4900 6100 4800
 Connection ~ 6000 4900
+$Comp
+L R R11
+U 1 1 5A935F18
+P 1100 1550
+F 0 "R11" V 1180 1550 50  0000 C CNN
+F 1 "0Ω" V 1100 1550 50  0000 C CNN
+F 2 "Resistors_SMD:R_0402" V 1030 1550 50  0001 C CNN
+F 3 "" H 1100 1550 50  0001 C CNN
+F 4 "DNP" V 1000 1550 60  0000 C CNN "Note"
+	1    1100 1550
+	-1   0    0    -1
+$EndComp
+Wire Wire Line
+	1100 1300 1100 1400
+$Comp
+L Test_Point TP3
+U 1 1 5A9367B6
+P 6900 5900
+F 0 "TP3" H 6900 6170 50  0000 C CNN
+F 1 "Setup" H 6900 6100 50  0000 C CNN
+F 2 "Measurement_Points:Measurement_Point_Round-SMD-Pad_Small" H 7100 5900 50  0001 C CNN
+F 3 "" H 7100 5900 50  0001 C CNN
+	1    6900 5900
+	0    1    1    0
+$EndComp
+$Comp
+L Conn_02x05_Odd_Even P1
+U 1 1 5A9380E9
+P 4800 6200
+F 0 "P1" H 4850 6500 50  0000 C CNN
+F 1 "SWD" H 4850 5900 50  0000 C CNN
+F 2 "Pin_Headers:Pin_Header_Straight_2x05_Pitch1.27mm_SMD" H 4800 6200 50  0001 C CNN
+F 3 "" H 4800 6200 50  0001 C CNN
+	1    4800 6200
+	1    0    0    -1
+$EndComp
 $EndSCHEMATC

Commit message: Update to KiCad 5.0 nightly
Hooray, new stuff!  The STM32 symbol is a reasonable size now!  We have
a sym-lib-table!  Everything is great, and I'm excited!

The board's a bit of a mess though, as the silkscreen needs to be laid
out nicely.  Oh well, details.
Parts:
- removed C10, C3, C4, C5, C6, C7, C8: 0.1μF, Capacitors_SMD:C_0402, symbol C
- removed C9: 1μF, Capacitors_SMD:C_0402, symbol C
- removed D4: Status, LEDs:LED_0603, symbol LED
- removed P1: SWD, Pin_Headers:Pin_Header_Straight_2x05_Pitch1.27mm_SMD, symbol Conn_02x05_Odd_Even
- removed R1, R3, R4: 2kΩ, Resistors_SMD:R_0402, symbol R
- removed R10: 220Ω, Resistors_SMD:R_0402, symbol R
- removed R11: 0Ω, Resistors_SMD:R_0402, symbol R
- removed R2, R5, R6: 10kΩ, Resistors_SMD:R_0402, symbol R
- removed SW2: Setup, Buttons_Switches_SMD:SW_SPST_PTS810, symbol SW_Push
- removed TP3: Setup, Measurement_Points:Measurement_Point_Round-SMD-Pad_Small, symbol Test_Point
- removed U2: STM32F072C8Ux, Housings_DFN_QFN:QFN-48-1EP_7x7mm_Pitch0.5mm, symbol STM32F072C8Ux
- added C3, C4, C5, C6, C7, C8: 0.1μF, Capacitor_SMD:C_0402_1005Metric, symbol Device:C
- added C9: 1μF, Capacitor_SMD:C_0402_1005Metric, symbol Device:C
- added D4: Status, LED_SMD:LED_0603_1608Metric, symbol Device:LED
- added JP1: Boot, Jumper:SolderJumper-2_P1.3mm_Open_RoundedPad1.0x1.5mm, symbol Jumper:SolderJumper_2_Open
- added P1: SWD, Connector_PinHeader_1.27mm:PinHeader_2x05_P1.27mm_Vertical_SMD, symbol Connector:Conn_ARM_JTAG_SWD_10
- added R1, R3, R4: 2kΩ, Resistor_SMD:R_0402_1005Metric, symbol Device:R
- added R10: 220Ω, Resistor_SMD:R_0402_1005Metric, symbol Device:R
- added R2, R6: 10kΩ, Resistor_SMD:R_0402_1005Metric, symbol Device:R
- added SW2: Setup, Button_Switch_SMD:SW_SPST_PTS810, symbol Switch:SW_Push
- added TP3: Setup, TestPoint:TestPoint_Pad_D1.5mm, symbol Connector:Test_Point
- added U2: STM32F072C8Ux, Package_DFN_QFN:QFN-48-1EP_7x7mm_P0.5mm_EP5.15x5.15mm, symbol MCU_ST_STM32F0:STM32F072C8Ux
Connections:
- net labels added: +3V3
- net labels removed: +3.3V
- wire segments 69 -> 87
- no-connect marks 30 -> 29

Commit message: Update footprints
Hooray for new, better footprints~!
Parts:
- U2: footprint Package_DFN_QFN:QFN-48-1EP_7x7mm_P0.5mm_EP5.15x5.15mm -> Package_DFN_QFN:QFN-48-1EP_7x7mm_P0.5mm_EP5.6x5.6mm
Changed lines of the file:
@@
 F 0 "U2" H 5350 4750 50  0000 C CNN
 F 1 "STM32F072C8Ux" H 6450 4750 50  0000 C CNN
-F 2 "Package_DFN_QFN:QFN-48-1EP_7x7mm_P0.5mm_EP5.15x5.15mm" H 5300 1900 50  0001 R CNN
+F 2 "Package_DFN_QFN:QFN-48-1EP_7x7mm_P0.5mm_EP5.6x5.6mm" H 5300 1900 50  0001 R CNN
 F 3 "http://www.st.com/st-web-ui/static/active/en/resource/technical/document/datasheet/DM00090510.pdf" H 5900 3300 50  0001 C CNN
 	1    5900 3300
